Commit message: updated model and configuration to SLAM correctly - add a wall to turtlebot3_house to make it a closed space - modified physical parameter of robot model to improve precision, also modified cartographer configuration - rename robot_footprint part to conventional name base_link

File: src/slambot/model/model.xacro (robot description, xacro)
@@ -29,8 +29,8 @@
   </ros2_control>
   <!-- 机器人本体结构 -->
-  <link name="robot_footprint"></link>
-  <joint name="robot_footprint_joint" type="fixed">
+  <link name="base_link"></link>
+  <joint name="base_link_joint" type="fixed">
     <origin xyz="0 0 0" rpy="0 0 0" />
-    <parent link="robot_footprint"/>
+    <parent link="base_link"/>
     <child link="chassis" />
   </joint>
@@ -153,5 +153,5 @@
     <axis xyz="0 1 0" rpy="0 0 0"/>
     <limit effort="10000" velocity="1000"/>
-    <dynamics damping="1.0" friction="1.0"/>
+    <dynamics damping="0.01" friction="0.1"/>
   </joint>
   <gazebo reference="left_wheel">
@@ -183,5 +183,5 @@
     <axis xyz="0 1 0" rpy="0 0 0"/>
     <limit effort="10000" velocity="1000"/>
-    <dynamics damping="1.0" friction="1.0"/>
+    <dynamics damping="0.01" friction="0.1"/>
   </joint>
   <gazebo reference="right_wheel">
@@ -269,6 +269,6 @@
             <samples>720</samples>
             <resolution>1</resolution>
-            <min_angle>-1.570796</min_angle>
-            <max_angle>1.570796</max_angle>
+            <min_angle>-2.356194</min_angle> <!-- -135° -->
+            <max_angle>2.356194</max_angle>  <!-- +135° -->
           </horizontal>
         </scan>
